Commit message: conversions to obj

File: husky_description/urdf/husky.urdf (robot description, URDF)
Before this commit: robot husky, 16 links, 15 joints
Links:
- link base_link: geometry collision box size=0.7899200000000001 0.5709 0.10375; collision box size=0.9874 0.5709 0.12375
- link front_bumper_link: geometry visual mesh filename=package://husky_description/meshes/bumper.mtl
- link front_left_wheel: geometry collision cylinder length=0.1143 radius=0.1651; visual mesh filename=package://husky_description/meshes/wheel.mtl
- link front_right_wheel: geometry collision cylinder length=0.1143 radius=0.1651; visual mesh filename=package://husky_description/meshes/wheel.mtl
- link rear_bumper_link: geometry visual mesh filename=package://husky_description/meshes/bumper.mtl
- link rear_left_wheel: geometry collision cylinder length=0.1143 radius=0.1651; visual mesh filename=package://husky_description/meshes/wheel.mtl
- link rear_right_wheel: geometry collision cylinder length=0.1143 radius=0.1651; visual mesh filename=package://husky_description/meshes/wheel.mtl
- link top_chassis_link: geometry visual mesh filename=package://husky_description/meshes/top_chassis.mtl
- link top_plate_link: geometry collision mesh filename=package://husky_description/meshes/top_plate.obj; visual mesh filename=package://husky_description/meshes/top_plate.mtl
- link user_rail_link: geometry visual mesh filename=package://husky_description/meshes/user_rail.mtl

Commit message: stuff I missed last time

File: husky_description/urdf/husky.urdf (robot description, URDF)
Before this commit: robot husky, 16 links, 15 joints
Links:
- link front_bumper_link: geometry visual mesh filename=package://husky_description/meshes/bumper.dae
- link rear_bumper_link: geometry visual mesh filename=package://husky_description/meshes/bumper.dae

Commit message: [feature] get nav to work!

File: husky_description/urdf/husky.urdf (robot description, URDF)
Before this commit: robot husky, 16 links, 15 joints
Links:
- link top_plate_link: geometry collision mesh filename=package://husky_description/meshes/top_plate.obj; visual mesh filename=package://husky_description/meshes/russ_test_obj.obj
